File: 00-produccion-pcbs/1-versiones-profes/grupo-02/secuenciador-02-v03/secuenciador-02-v03.kicad_pcb (KiCad board)
At the start: 2 copper layers, 100 x 100 mm, 55 parts, among them J10 AudioJack2_SwitchT, J11 AudioJack2_SwitchT, J12 AudioJack2_SwitchT, J13 AudioJack2_SwitchT, J14 AudioJack2_SwitchT, J2 Barrel_Jack_Switch, J4 Barrel_Jack_Switch, J6 AudioJack2_SwitchT, J7 AudioJack2_SwitchT, J8 AudioJack2_SwitchT, J9 AudioJack2_SwitchT, Q1 BC548, Q10 PN2222A, Q3 PN2222A, Q4 PN2222A, Q5 PN2222A, Q6 PN2222A, Q7 PN2222A, Q8 PN2222A, Q9 PN2222A, SW4 SW_SPDT, U2 4015, U4 L7805

Commit message: terminado g02
Parts:
- added H1: M3, MountingHole:MountingHole_3.2mm_M3, F.Cu at (148.0, 59.0)
- added H2: M3, MountingHole:MountingHole_3.2mm_M3, F.Cu at (183.0, 59.0)
- added H3: M3, MountingHole:MountingHole_3.2mm_M3, F.Cu at (118.0, 130.0)
- added H4: M3, MountingHole:MountingHole_3.2mm_M3, F.Cu at (211.0, 128.0)
- added R13: 100k, Resistor_THT:R_Axial_DIN0207_L6.3mm_D2.5mm_P10.16mm_Horizontal, F.Cu at (189.2, 151.0)
- added R23: 1k, Resistor_THT:R_Axial_DIN0207_L6.3mm_D2.5mm_P10.16mm_Horizontal, B.Cu at (200.8, 78.0)
- added R24: 1k, Resistor_THT:R_Axial_DIN0207_L6.3mm_D2.5mm_P10.16mm_Horizontal, B.Cu at (201.2, 99.6)
- added R25: 1k, Resistor_THT:R_Axial_DIN0207_L6.3mm_D2.5mm_P10.16mm_Horizontal, B.Cu at (201.3, 122.7)
- added R26: 1k, Resistor_THT:R_Axial_DIN0207_L6.3mm_D2.5mm_P10.16mm_Horizontal, B.Cu at (201.2, 133.2)
- added R27: 1k, Resistor_THT:R_Axial_DIN0207_L6.3mm_D2.5mm_P10.16mm_Horizontal, B.Cu at (129.0, 146.5)
- added R28: 1k, Resistor_THT:R_Axial_DIN0207_L6.3mm_D2.5mm_P10.16mm_Horizontal, B.Cu at (129.0, 123.2)
- added R29: 1k, Resistor_THT:R_Axial_DIN0207_L6.3mm_D2.5mm_P10.16mm_Horizontal, B.Cu at (129.0, 100.2)
- added R30: 1k, Resistor_THT:R_Axial_DIN0207_L6.3mm_D2.5mm_P10.16mm_Horizontal, B.Cu at (129.1, 77.0)
- Q1, Q10, Q3, Q4, Q5, Q6, Q7, Q8, Q9: footprint Package_TO_SOT_THT:TO-92_Inline -> Package_TO_SOT_THT:TO-92_Inline_Wide
- moved Q6 0.19 mm to (195.3, 139.5)
- moved Q3 0.17 mm to (195.2, 70.1)
Connections:
- J10 pad 3: Net-(U2A-D) -> Net-(J10-Pad3)
- J11 pad 3: Net-(U2A-Q1) -> Net-(J11-Pad3)
- J12 pad 3: Net-(U2A-Q2) -> Net-(J12-Pad3)
- J13 pad 3: Net-(U2A-Q3) -> Net-(J13-Pad3)
- J14 pad 3: Net-(U2A-Q4) -> Net-(J14-Pad3)
- J7 pad 3: Net-(U2B-Q1) -> Net-(J7-Pad3)
- J8 pad 3: Net-(U2B-Q2) -> Net-(J8-Pad3)
- J9 pad 3: Net-(U2B-Q3) -> Net-(J9-Pad3)
Routing:
- net Net-(U2A-CP): track 94.8 -> 110.0 mm, vias 1 -> 2
- net Net-(U2A-Q2): track 77.1 -> 62.1 mm
- net Net-(U2A-Q1): track 98.1 -> 83.8 mm
- net Net-(U2A-Q3): track 60.0 -> 45.9 mm
- net Net-(U2A-D): track 104.1 -> 92.8 mm
- net Net-(J7-Pad3): track 0.00 -> 7.82 mm
- net Net-(J11-Pad3): track 0.00 -> 7.47 mm
- net Net-(J9-Pad3): track 0.00 -> 7.15 mm
- net Net-(J12-Pad3): track 0.00 -> 7.13 mm
- net Net-(J13-Pad3): track 0.00 -> 7.07 mm
- net Net-(J8-Pad3): track 0.00 -> 7.07 mm
- net Net-(J10-Pad3): track 0.00 -> 6.93 mm
- net Net-(J14-Pad3): track 0.00 -> 6.90 mm
- net Net-(U2A-Q4): track 119.4 -> 123.9 mm
- net Net-(U2B-Q3): track 60.6 -> 63.8 mm
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