File: 00-produccion-pcbs/1-versiones-profes/grupo-02/secuenciador-02-v03/secuenciador-02-v03.kicad_sch (KiCad schematic)
At the start: 55 parts, among them J10 AudioJack2_SwitchT, J11 AudioJack2_SwitchT, J12 AudioJack2_SwitchT, J13 AudioJack2_SwitchT, J14 AudioJack2_SwitchT, J2 Barrel_Jack_Switch, J4 Barrel_Jack_Switch, J6 AudioJack2_SwitchT, J7 AudioJack2_SwitchT, J8 AudioJack2_SwitchT, J9 AudioJack2_SwitchT, Q1 BC548, Q10 PN2222A, Q3 PN2222A, Q4 PN2222A, Q5 PN2222A, Q6 PN2222A, Q7 PN2222A, Q8 PN2222A, Q9 PN2222A, SW4 SW_SPDT, U2 4015, U4 L7805

Commit message: terminado g02
Parts:
- added H1, H2, H3, H4: M3, MountingHole:MountingHole_3.2mm_M3, symbol Mechanical:MountingHole
- added R13: 100k, Resistor_THT:R_Axial_DIN0207_L6.3mm_D2.5mm_P10.16mm_Horizontal, symbol Device:R
- added R23, R24, R25, R26, R27, R28, R29, R30: 1k, Resistor_THT:R_Axial_DIN0207_L6.3mm_D2.5mm_P10.16mm_Horizontal, symbol Device:R
- Q1, Q10, Q3, Q4, Q5, Q6, Q7, Q8, Q9: footprint Package_TO_SOT_THT:TO-92_Inline -> Package_TO_SOT_THT:TO-92_Inline_Wide
Connections:
- net GND: now also R13.1
- net at R16.2, U2.12 (Q2): now also R24.1; no longer J8.3
- net at J6.3, U2.1 (CP), U2.9 (CP): now also R13.2
- net at R17.2, U2.11 (Q3): now also R25.1; no longer J9.3
- net at R15.2, U2.13 (Q1): now also R23.1; no longer J7.3
- net at R18.2, U2.2 (Q4), U2.7 (D): now also R26.1; no longer J10.3
- net at R20.2, U2.4 (Q2): now also R28.1; no longer J12.3
- net at R21.2, U2.3 (Q3): now also R29.1; no longer J13.3
- net at R2.2, R22.2, U2.10 (Q4): now also R30.1; no longer J14.3
- net at R19.2, U2.5 (Q1): now also R27.1; no longer J11.3
- new net: J12.3, R28.2
- new net: J14.3, R30.2
- new net: J9.3, R25.2
- new net: J10.3, R26.2
- new net: J11.3, R27.2
- new net: J7.3, R23.2
- new net: J13.3, R29.2
- new net: J8.3, R24.2
