File: 00-produccion-pcbs/1-versiones-profes/grupo-03/g-03-osc-02-rev-a/g-03-osc-02-rev-a.kicad_pcb (KiCad board)
At the start: 2 copper layers, 100 x 70 mm, 29 parts, among them J1 Barrel_Jack_Switch, J3 Barrel_Jack_Switch, J4 AudioJack2_SwitchT, J5 Conn_01x03_Pin, SW3 SW_SPDT, U1 4017, U2 4046, U3 40106, U4 L7805

Commit message: añadido g-03-02
Parts:
- removed C1: 10uF, Capacitor_THT:CP_Radial_D5.0mm_P2.00mm
- added C8: 10u, Capacitor_THT:CP_Radial_D4.0mm_P2.00mm, F.Cu at (132.0, 106.0)
- C3: value 4.7uF -> 4u7
- C7: value 10uF -> 1u; footprint Capacitor_THT:CP_Radial_D5.0mm_P2.00mm -> Capacitor_THT:C_Disc_D5.0mm_W2.5mm_P2.50mm
- moved C7 44.5 mm to (155.0, 77.5), turned to 90 degrees
Connections:
- J4 pad 1: Net-(C7-Pad2) -> GND
- J4 pad 2: GND -> unconnected-(J4-Pad2)
- J4 pad 3: unconnected-(J4-Pad3) -> Net-(C7-Pad2)
Routing:
- net GND: track 0.00 -> 45.8 mm, vias 0 -> 2
- net Net-(C7-Pad2): track 45.3 -> 9.60 mm, vias 2 -> 0
- net Net-(U1-CLK): track 71.1 -> 85.1 mm
- net Net-(U2-VCOin): track 74.1 -> 77.8 mm
- net Net-(C8-Pad1): track 11.2 -> 13.9 mm
Other:
- board text added: "g-03-osc-02-rev-a"
