File: 00-produccion-pcbs/1-versiones-profes/grupo-03/g-03-osc-02-rev-a/g-03-osc-02-rev-a.kicad_sch (KiCad schematic)
At the start: 29 parts, among them J1 Barrel_Jack_Switch, J3 Barrel_Jack_Switch, J4 AudioJack2_SwitchT, J5 Conn_01x03_Pin, SW3 SW_SPDT, U1 4017, U2 4046, U3 40106, U4 L7805

Commit message: añadido g-03-02
Parts:
- removed C1: 10uF, Capacitor_THT:CP_Radial_D5.0mm_P2.00mm, symbol Device:C
- added C8: 10u, Capacitor_THT:CP_Radial_D4.0mm_P2.00mm, symbol Device:C_Polarized
- C3: value 4.7uF -> 4u7
- C7: value 10uF -> 1u; footprint Capacitor_THT:CP_Radial_D5.0mm_P2.00mm -> Capacitor_THT:C_Disc_D5.0mm_W2.5mm_P2.50mm
Connections:
- net GND: now also J4.1, C8.2; no longer J4.2
- net at R2.2: now also C8.1
- net at C7.2: now also J4.3; no longer J4.1
Other:
- moved on the sheet: J4
